File: pi_hat/bibby_pi_hat/bibby_pi_hat.kicad_pcb (KiCad board)
At the start: 2 copper layers, 65 x 56 mm, 21 parts, among them J1 GPIO, J2 Conn_01x10, U1 MAX31865xAP, U2 H11AA1

Commit message: corrections on pi_hat. DRDYn from max chip went to wrong pin and two grounds of max chip weren't connected.
Connections:
- U1 pad 16: /GPIO14/TXD0/CS -> /GPIO8/SPI0.CE0
Routing:
- net /GPIO14/TXD0/CS: track 49.3 -> 0.00 mm
- net /GPIO8/SPI0.CE0: track 0.00 -> 27.5 mm
- net /GPIO11/SPI0.SCLK: track 22.7 -> 24.7 mm
- net /GPIO10/SPI0.MOSI: track 28.0 -> 29.1 mm
Changed lines of the file:
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@@
 			(layers "F.Cu" "F.Mask" "F.Paste")
 			(roundrect_rratio 0.25)
-			(net "/GPIO14{slash}TXD0{slash}CS")
+			(net "/GPIO8{slash}SPI0.CE0")
 			(pinfunction "~{CS}_16")
 			(pintype "input")
@@
 	)
 	(segment
-		(start 131.23 48.77)
-		(end 132.3848 49.9248)
+		(start 148.357632 62.857632)
+		(end 148.357632 61.392368)
 		(width 0.2032)
 		(layer "F.Cu")
@@
 	)
 	(segment
-		(start 149.6924 63.968646)
-		(end 150.884754 65.161)
+		(start 151.76 65.161)
+		(end 150.661 65.161)
 		(width 0.2032)
 		(layer "F.Cu")
@@
 	)
 	(segment
-		(start 136.890064 49.9248)
-		(end 149.6924 62.727136)
+		(start 132.3848 49.9248)
+		(end 136.890064 49.9248)
 		(width 0.2032)
 		(layer "F.Cu")
@@
 	)
 	(segment
-		(start 150.884754 65.161)
-		(end 151.76 65.161)
+		(start 151.76 65.161)
+		(end 150.884754 65.161)
 		(width 0.2032)
 		(layer "F.Cu")
@@
 	)
 	(segment
-		(start 149.6924 62.727136)
-		(end 149.6924 63.968646)
+		(start 131.23 48.77)
+		(end 132.3848 49.9248)
 		(width 0.2032)
 		(layer "F.Cu")
@@
 	)
 	(segment
-		(start 132.3848 49.9248)
-		(end 136.890064 49.9248)
+		(start 136.890064 49.9248)
+		(end 148.357632 61.392368)
 		(width 0.2032)
 		(layer "F.Cu")
@@
 	)
 	(segment
-		(start 150.0988 62.999782)
-		(end 150.5052 63.406182)
+		(start 150.661 65.161)
+		(end 148.357632 62.857632)
 		(width 0.2032)
 		(layer "F.Cu")
-		(net "/GPIO11{slash}SPI0.SCLK")
+		(net "/GPIO10{slash}SPI0.MOSI")
 	)
 	(segment
-		(start 150.5052 64.206199)
-		(end 150.810001 64.511)
+		(start 148.895 62.645)
+		(end 148.895 61.355)
 		(width 0.2032)
 		(layer "F.Cu")
@@
 	)
 	(segment
-		(start 150.0988 62.5588)
-		(end 150.0988 62.999782)
+		(start 150.549001 64.25)
+		(end 150.810001 64.511)
 		(width 0.2032)
 		(layer "F.Cu")
@@
 	)
 	(segment
-		(start 150.810001 64.511)
-		(end 151.76 64.511)
+		(start 150.761 64.511)
+		(end 148.895 62.645)
 		(width 0.2032)
 		(layer "F.Cu")
@@
 	)
 	(segment
-		(start 150.5052 63.406182)
-		(end 150.5052 64.206199)
+		(start 150.549001 64.25)
+		(end 150.0988 63.799799)
 		(width 0.2032)
 		(layer "F.Cu")
@@
 	)
 	(segment
-		(start 136.31 48.77)
-		(end 150.0988 62.5588)
+		(start 150.810001 64.511)
+		(end 151.76 64.511)
 		(width 0.2032)
 		(layer "F.Cu")
@@
 	)
 	(segment
-		(start 148.171123 56.146877)
-		(end 146.903343 56.146877)
+		(start 136.31 48.77)
+		(end 148.895 61.355)
 		(width 0.2032)
 		(layer "F.Cu")
-		(net "/GPIO14{slash}TXD0{slash}CS")
+		(net "/GPIO11{slash}SPI0.SCLK")
 	)
 	(segment
-		(start 138.178466 47.422)
-		(end 137.4648 46.708334)
+		(start 151.76 64.511)
+		(end 150.761 64.511)
 		(width 0.2032)
 		(layer "F.Cu")
-		(net "/GPIO14{slash}TXD0{slash}CS")
-	)
-	(segment
-		(start 151.76 63.861)
-		(end 152.709999 63.861)
-		(width 0.2032)
-		(layer "F.Cu")
-		(net "/GPIO14{slash}TXD0{slash}CS")
+		(net "/GPIO11{slash}SPI0.SCLK")
 	)
 	(segment
-		(start 140.132 49.375534)
-		(end 140.132 48.184)
+		(start 151.76 63.211)
+		(end 150.211 63.211)
 		(width 0.2032)
 		(layer "F.Cu")
-		(net "/GPIO14{slash}TXD0{slash}CS")
+		(net "/GPIO9{slash}SPI0.MISO")
 	)
 	(segment
-		(start 146.903343 56.146877)
-		(end 140.132 49.375534)
+		(start 149.444 62.444)
+		(end 149.444 61.306)
 		(width 0.2032)
 		(layer "F.Cu")
-		(net "/GPIO14{slash}TXD0{slash}CS")
+		(net "/GPIO9{slash}SPI0.MISO")
 	)
 	(segment
-		(start 153.0148 63.556199)
-		(end 153.0148 60.990554)
+		(start 137.4648 48.291666)
+		(end 136.788334 47.6152)
 		(width 0.2032)
 		(layer "F.Cu")
-		(net "/GPIO14{slash}TXD0{slash}CS")
+		(net "/GPIO9{slash}SPI0.MISO")
 	)
 	(segment
-		(start 137.4648 46.708334)
-		(end 137.4648 45.751666)
+		(start 136.788334 47.6152)
+		(end 134.9248 47.6152)
 		(width 0.2032)
 		(layer "F.Cu")
-		(net "/GPIO14{slash}TXD0{slash}CS")
+		(net "/GPIO9{slash}SPI0.MISO")
 	)
 	(segment
-		(start 152.709999 63.861)
-		(end 153.0148 63.556199)
+		(start 137.4648 49.3268)
+		(end 137.4648 48.291666)
 		(width 0.2032)
 		(layer "F.Cu")
-		(net "/GPIO14{slash}TXD0{slash}CS")
+		(net "/GPIO9{slash}SPI0.MISO")
 	)
 	(segment
-		(start 117.1448 45.0752)
-		(end 115.99 46.23)
+		(start 150.211 63.211)
+		(end 149.444 62.444)
 		(width 0.2032)
 		(layer "F.Cu")
-		(net "/GPIO14{slash}TXD0{slash}CS")
+		(net "/GPIO9{slash}SPI0.MISO")
 	)
 	(segment
-		(start 137.4648 45.751666)
-		(end 136.788334 45.0752)
+		(start 134.9248 47.6152)
+		(end 133.77 48.77)
 		(width 0.2032)
 		(layer "F.Cu")
-		(net "/GPIO14{slash}TXD0{slash}CS")
+		(net "/GPIO9{slash}SPI0.MISO")
 	)
 	(segment
-		(start 139.37 47.422)
-		(end 138.178466 47.422)
+		(start 149.444 61.306)
+		(end 137.4648 49.3268)
 		(width 0.2032)
 		(layer "F.Cu")
-		(net "/GPIO14{slash}TXD0{slash}CS")
+		(net "/GPIO9{slash}SPI0.MISO")
 	)
 	(segment
-		(start 136.788334 45.0752)
-		(end 117.1448 45.0752)
+		(start 116.002 74.6)
+		(end 116.002 77.855)
 		(width 0.2032)
 		(layer "F.Cu")
-		(net "/GPIO14{slash}TXD0{slash}CS")
+		(net "Net-(R5-Pad2)")
 	)
 	(segment
-		(start 140.132 48.184)
-		(end 139.37 47.422)
+		(start 113.208 69.266)
+		(end 116.002 72.06)
 		(width 0.2032)
 		(layer "F.Cu")
-		(net "/GPIO14{slash}TXD0{slash}CS")
+		(net "Net-(R6-Pad2)")
 	)
 	(segment
-		(start 153.0148 60.990554)
-		(end 148.171123 56.146877)
+		(start 116.002 72.06)
+		(end 116.002 72.775)
 		(width 0.2032)
 		(layer "F.Cu")
-		(net "/GPIO14{slash}TXD0{slash}CS")
+		(net "Net-(R6-Pad2)")
 	)
 	(segment
-		(start 137.4648 48.291666)
-		(end 137.4648 49.3268)
-		(width 0.2032)
+		(start 108.37 46.23)
+		(end 110.91 46.23)
+		(width 0.3048)
 		(layer "F.Cu")
-		(net "/GPIO9{slash}SPI0.MISO")
+		(net "+5V")
 	)
 	(segment
-		(start 150.5052 62.3672)
-		(end 150.5052 62.831446)
+		(start 137.502 47.422)
+		(end 136.31 46.23)
 		(width 0.2032)
 		(layer "F.Cu")
-		(net "/GPIO9{slash}SPI0.MISO")
+		(net "/GPIO8{slash}SPI0.CE0")
 	)
 	(segment
-		(start 150.884754 63.211)
-		(end 151.76 63.211)
+		(start 140.132 48.184)
+		(end 139.37 47.422)
 		(width 0.2032)
 		(layer "F.Cu")
-		(net "/GPIO9{slash}SPI0.MISO")
+		(net "/GPIO8{slash}SPI0.CE0")
 	)
 	(segment
-		(start 133.77 48.77)
-		(end 134.9248 47.6152)
+		(start 152.709999 63.861)
+		(end 153.0148 63.556199)
 		(width 0.2032)
 		(layer "F.Cu")
-		(net "/GPIO9{slash}SPI0.MISO")
+		(net "/GPIO8{slash}SPI0.CE0")
 	)
 	(segment
-		(start 137.4648 49.3268)
-		(end 150.5052 62.3672)
+		(start 153.0148 63.556199)
+		(end 153.0148 60.990554)
 		(width 0.2032)
 		(layer "F.Cu")
-		(net "/GPIO9{slash}SPI0.MISO")
+		(net "/GPIO8{slash}SPI0.CE0")
 	)
 	(segment
-		(start 136.788334 47.6152)
-		(end 137.4648 48.291666)
+		(start 139.37 47.422)
+		(end 137.502 47.422)
 		(width 0.2032)
 		(layer "F.Cu")
-		(net "/GPIO9{slash}SPI0.MISO")
+		(net "/GPIO8{slash}SPI0.CE0")
 	)
 	(segment
-		(start 134.9248 47.6152)
-		(end 136.788334 47.6152)
+		(start 151.76 63.861)
+		(end 152.709999 63.861)
 		(width 0.2032)
 		(layer "F.Cu")
-		(net "/GPIO9{slash}SPI0.MISO")
+		(net "/GPIO8{slash}SPI0.CE0")
 	)
 	(segment
-		(start 150.5052 62.831446)
-		(end 150.884754 63.211)
+		(start 153.0148 60.990554)
+		(end 148.171123 56.146877)
 		(width 0.2032)
 		(layer "F.Cu")
-		(net "/GPIO9{slash}SPI0.MISO")
+		(net "/GPIO8{slash}SPI0.CE0")
 	)
 	(segment
-		(start 116.002 74.6)
-		(end 116.002 77.855)
+		(start 140.132 49.375534)
+		(end 140.132 48.184)
 		(width 0.2032)
 		(layer "F.Cu")
-		(net "Net-(R5-Pad2)")
+		(net "/GPIO8{slash}SPI0.CE0")
 	)
 	(segment
-		(start 113.208 69.266)
-		(end 116.002 72.06)
+		(start 148.171123 56.146877)
+		(end 146.903343 56.146877)
 		(width 0.2032)
 		(layer "F.Cu")
-		(net "Net-(R6-Pad2)")
+		(net "/GPIO8{slash}SPI0.CE0")
 	)
 	(segment
-		(start 116.002 72.06)
-		(end 116.002 72.775)
+		(start 146.903343 56.146877)
+		(end 140.132 49.375534)
 		(width 0.2032)
 		(layer "F.Cu")
-		(net "Net-(R6-Pad2)")
-	)
-	(segment
-		(start 108.37 46.23)
-		(end 110.91 46.23)
-		(width 0.3048)
-		(layer "F.Cu")
-		(net "+5V")
+		(net "/GPIO8{slash}SPI0.CE0")
 	)
 	(zone
