File: pi_hat/bibby_pi_hat/bibby_pi_hat.kicad_sch (KiCad schematic)
At the start: 17 parts, among them J1 GPIO, J2 Conn_01x10, U1 MAX31865xAP, U2 H11AA1

Commit message: corrections on pi_hat. DRDYn from max chip went to wrong pin and two grounds of max chip weren't connected.
Connections:
- net GPIO14/TXD0/CS: no longer U1.16 (~{CS})
- net GPIO8/SPI0.CE0: now also U1.16 (~{CS})
Changed lines of the file:
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@@
 		)
 	)
-	(label "GPIO14{slash}TXD0{slash}CS"
+	(label "GPIO8{slash}SPI0.CE0"
 		(at 137.16 62.23 0)
 		(effects
